Commit message: Integrated manipulator into sim

File: micro_g_description/xacro/target/config.xacro (robot description, xacro)
@@ -1,4 +1,4 @@
 <?xml version="1.0"?>
-<robot name="target_testing" xmlns:xacro="http://ros.org/wiki/xacro">
+<robot name="target" xmlns:xacro="http://ros.org/wiki/xacro">
   <!-- Arguments -->
   <xacro:arg name="prefix" default="" />
@@ -10,15 +10,13 @@
   <xacro:property name="use_sim" value="$(arg use_sim)" />
   <link name="base_footprint" />
-  <!-- Import target macro -->
+  <!-- Imports -->
   <xacro:include filename="$(find ${description_package})/xacro/target/urdf.xacro" />
-  <xacro:target_urdf
-    parent="base_footprint"
-    prefix="${prefix}">
-    <origin xyz="0 0 1.0" rpy="0 0 0" />
+  <xacro:target_urdf parent="base_footprint" prefix="${prefix}">
+    <origin xyz="0.3 0 0.2" rpy="0 0 0" />
   </xacro:target_urdf>
   <!-- Import the Gazebo macro -->
-  <xacro:if value="$(arg use_sim)">
+  <xacro:if value="${use_sim}">
     <xacro:include filename="$(find ${description_package})/xacro/target/gazebo.xacro" />
-    <xacro:target_gazebo reference="$(arg prefix)target" />
+    <xacro:target_gazebo />
   </xacro:if>
 </robot>

File: micro_g_description/xacro/target/gazebo.xacro (robot description, xacro)
@@ -7,5 +7,5 @@
         filename="ignition-gazebo-velocity-control-system"
         name="ignition::gazebo::systems::VelocityControl">
-        <initial_linear>0.2 0 0</initial_linear>
+        <initial_linear>0 0 0</initial_linear>
         <initial_angular>0 0 0</initial_angular>
       </plugin>

File: micro_g_description/xacro/target/urdf.xacro (robot description, xacro)
@@ -2,5 +2,5 @@
 <robot xmlns:xacro="http://ros.org/wiki/xacro">
   <xacro:macro name="target_urdf" params="prefix parent *origin">
-    <link name="${prefix}target">
+    <link name="${prefix}target_link">
       <inertial>
         <mass value="0.0001" />
@@ -16,5 +16,5 @@
       <visual>
         <geometry>
-          <box size="0.5 0.5 0.5" />
+          <box size="0.02 0.02 0.02" />
         </geometry>
         <xacro:insert_block name="origin" />
@@ -22,5 +22,5 @@
       <collision>
         <geometry>
-          <box size="0.5 0.5 0.5" />
+          <box size="0.02 0.02 0.02" />
         </geometry>
         <xacro:insert_block name="origin" />
@@ -29,14 +29,6 @@
     <joint name="${prefix}base_footprint_joint" type="fixed">
       <parent link="${prefix}base_footprint" />
-      <child link="${prefix}target" />
+      <child link="${prefix}target_link" />
     </joint>
-    <gazebo reference="${prefix}target">
-      <plugin
-        filename="gz-sim-velocity-control-system"
-        name="gz::sim::systems::VelocityControl">
-        <initial_linear>0.2 0 0</initial_linear>
-        <initial_angular>0 0 0</initial_angular>
-      </plugin>
-    </gazebo>
   </xacro:macro>
 </robot>
