Commit message: Fixed launch bugs and added rviz configuration

File: micro_g_description/xacro/px100/config.xacro (robot description, xacro)
@@ -3,6 +3,6 @@
   <!-- Arguments -->
   <xacro:arg name="prefix" default="" />
-  <xacro:arg name="use_sim" default="true" />
-  <xacro:arg name="use_fake_hardware" default="true" />
+  <xacro:arg name="use_sim" default="false" />
+  <xacro:arg name="use_fake_hardware" default="false" />
   <xacro:arg name="description_package" default="micro_g_description" />
   <!-- Properties -->
@@ -16,4 +16,7 @@
   <xacro:include filename="$(find ${description_package})/xacro/px100/urdf.xacro" />
   <xacro:include filename="$(find ${description_package})/xacro/px100/ros2_control.xacro" />
+  <xacro:px100_urdf prefix="${prefix}" parent="base_footprint" use_sim="${use_sim}">
+    <origin xyz="0 0 0" rpy="0 0 0" />
+  </xacro:px100_urdf>
   <xacro:px100_system
     prefix="${prefix}"
@@ -21,6 +24,3 @@
     use_fake_hardware="${use_fake_hardware}"
   />
-  <xacro:px100_urdf prefix="${prefix}" parent="base_footprint" use_sim="${use_sim}">
-    <origin xyz="0 0 0" rpy="0 0 0" />
-  </xacro:px100_urdf>
 </robot>

File: micro_g_description/xacro/px100/ros2_control.xacro (robot description, xacro)
@@ -5,10 +5,10 @@
     <xacro:property name="pi_offset" value="0.00001" />
     <ros2_control name="XSHardwareInterface" type="system">
-      <xacro:if value="$(arg use_sim)">
+      <xacro:if value="${use_sim}">
         <hardware>
           <plugin>gz_ros2_control/GazeboSimSystem</plugin>
         </hardware>
       </xacro:if>
-      <xacro:unless value="$(arg use_sim)">
+      <xacro:unless value="${use_sim}">
         <hardware>
           <xacro:if value="${use_fake_hardware}">

File: micro_g_description/xacro/px100/urdf.xacro (robot description, xacro)
@@ -14,15 +14,15 @@
         <geometry>
           <mesh
-            filename="$(find interbotix_xsarm_descriptions)/meshes/px100_meshes/base.stl"
-            scale="0.001 0.001 0.001"
-          />
-        </geometry>
-        <material name="interbotix_black" />
-      </visual>
-      <collision>
-        <origin rpy="0 0 ${pi/2}" xyz="0 0 0" />
-        <geometry>
-          <mesh
-            filename="$(find interbotix_xsarm_descriptions)/meshes/px100_meshes/base.stl"
+            filename="file://$(find interbotix_xsarm_descriptions)/meshes/px100_meshes/base.stl"
+            scale="0.001 0.001 0.001"
+          />
+        </geometry>
+        <material name="interbotix_black" />
+      </visual>
+      <collision>
+        <origin rpy="0 0 ${pi/2}" xyz="0 0 0" />
+        <geometry>
+          <mesh
+            filename="file://$(find interbotix_xsarm_descriptions)/meshes/px100_meshes/base.stl"
             scale="0.001 0.001 0.001"
           />
@@ -47,5 +47,5 @@
         <geometry>
           <mesh
-            filename="$(find interbotix_xsarm_descriptions)/meshes/px100_meshes/shoulder.stl"
+            filename="file://$(find interbotix_xsarm_descriptions)/meshes/px100_meshes/shoulder.stl"
             scale="0.001 0.001 0.001" />
         </geometry>
@@ -56,5 +56,5 @@
         <geometry>
           <mesh
-            filename="$(find interbotix_xsarm_descriptions)/meshes/px100_meshes/shoulder.stl"
+            filename="file://$(find interbotix_xsarm_descriptions)/meshes/px100_meshes/shoulder.stl"
             scale="0.001 0.001 0.001"
           />
@@ -79,15 +79,15 @@
         <geometry>
           <mesh
-            filename="$(find interbotix_xsarm_descriptions)/meshes/px100_meshes/upper_arm.stl"
-            scale="0.001 0.001 0.001"
-          />
-        </geometry>
-        <material name="interbotix_black" />
-      </visual>
-      <collision>
-        <origin rpy="0 0 ${pi/2}" xyz="0 0 0" />
-        <geometry>
-          <mesh
-            filename="$(find interbotix_xsarm_descriptions)/meshes/px100_meshes/upper_arm.stl"
+            filename="file://$(find interbotix_xsarm_descriptions)/meshes/px100_meshes/upper_arm.stl"
+            scale="0.001 0.001 0.001"
+          />
+        </geometry>
+        <material name="interbotix_black" />
+      </visual>
+      <collision>
+        <origin rpy="0 0 ${pi/2}" xyz="0 0 0" />
+        <geometry>
+          <mesh
+            filename="file://$(find interbotix_xsarm_descriptions)/meshes/px100_meshes/upper_arm.stl"
             scale="0.001 0.001 0.001"
           />
@@ -112,15 +112,15 @@
         <geometry>
           <mesh
-            filename="$(find interbotix_xsarm_descriptions)/meshes/px100_meshes/forearm.stl"
-            scale="0.001 0.001 0.001"
-          />
-        </geometry>
-        <material name="interbotix_black" />
-      </visual>
-      <collision>
-        <origin rpy="0 0 ${pi/2}" xyz="0 0 0" />
-        <geometry>
-          <mesh
-            filename="$(find interbotix_xsarm_descriptions)/meshes/px100_meshes/forearm.stl"
+            filename="file://$(find interbotix_xsarm_descriptions)/meshes/px100_meshes/forearm.stl"
+            scale="0.001 0.001 0.001"
+          />
+        </geometry>
+        <material name="interbotix_black" />
+      </visual>
+      <collision>
+        <origin rpy="0 0 ${pi/2}" xyz="0 0 0" />
+        <geometry>
+          <mesh
+            filename="file://$(find interbotix_xsarm_descriptions)/meshes/px100_meshes/forearm.stl"
             scale="0.001 0.001 0.001"
           />
@@ -145,15 +145,15 @@
         <geometry>
           <mesh
-            filename="$(find interbotix_xsarm_descriptions)/meshes/px100_meshes/gripper.stl"
-            scale="0.001 0.001 0.001"
-          />
-        </geometry>
-        <material name="interbotix_black" />
-      </visual>
-      <collision>
-        <origin rpy="0 0 ${pi/2}" xyz="0 0 0" />
-        <geometry>
-          <mesh
-            filename="$(find interbotix_xsarm_descriptions)/meshes/px100_meshes/gripper.stl"
+            filename="file://$(find interbotix_xsarm_descriptions)/meshes/px100_meshes/gripper.stl"
+            scale="0.001 0.001 0.001"
+          />
+        </geometry>
+        <material name="interbotix_black" />
+      </visual>
+      <collision>
+        <origin rpy="0 0 ${pi/2}" xyz="0 0 0" />
+        <geometry>
+          <mesh
+            filename="file://$(find interbotix_xsarm_descriptions)/meshes/px100_meshes/gripper.stl"
             scale="0.001 0.001 0.001"
           />
@@ -190,5 +190,5 @@
         <geometry>
           <mesh
-            filename="$(find interbotix_xsarm_descriptions)/meshes/px100_meshes/gripper_prop.stl"
+            filename="file://$(find interbotix_xsarm_descriptions)/meshes/px100_meshes/gripper_prop.stl"
             scale="0.001 0.001 0.001" />
         </geometry>
@@ -199,5 +199,5 @@
         <geometry>
           <mesh
-            filename="$(find interbotix_xsarm_descriptions)/meshes/px100_meshes/gripper_prop.stl"
+            filename="file://$(find interbotix_xsarm_descriptions)/meshes/px100_meshes/gripper_prop.stl"
             scale="0.001 0.001 0.001"
           />
@@ -222,5 +222,5 @@
         <geometry>
           <mesh
-            filename="$(find interbotix_xsarm_descriptions)/meshes/px100_meshes/gripper_bar.stl"
+            filename="file://$(find interbotix_xsarm_descriptions)/meshes/px100_meshes/gripper_bar.stl"
             scale="0.001 0.001 0.001"
           />
@@ -232,5 +232,5 @@
         <geometry>
           <mesh
-            filename="$(find interbotix_xsarm_descriptions)/meshes/px100_meshes/gripper_bar.stl"
+            filename="file://$(find interbotix_xsarm_descriptions)/meshes/px100_meshes/gripper_bar.stl"
             scale="0.001 0.001 0.001"
           />
@@ -268,5 +268,5 @@
         <geometry>
           <mesh
-            filename="$(find interbotix_xsarm_descriptions)/meshes/px100_meshes/gripper_finger.stl"
+            filename="file://$(find interbotix_xsarm_descriptions)/meshes/px100_meshes/gripper_finger.stl"
             scale="0.001 0.001 0.001" />
         </geometry>
@@ -277,5 +277,5 @@
         <geometry>
           <mesh
-            filename="$(find interbotix_xsarm_descriptions)/meshes/px100_meshes/gripper_finger.stl"
+            filename="file://$(find interbotix_xsarm_descriptions)/meshes/px100_meshes/gripper_finger.stl"
             scale="0.001 0.001 0.001"
           />
@@ -300,5 +300,5 @@
         <geometry>
           <mesh
-            filename="$(find interbotix_xsarm_descriptions)/meshes/px100_meshes/gripper_finger.stl"
+            filename="file://$(find interbotix_xsarm_descriptions)/meshes/px100_meshes/gripper_finger.stl"
             scale="0.001 0.001 0.001"
           />
@@ -310,5 +310,5 @@
         <geometry>
           <mesh
-            filename="$(find interbotix_xsarm_descriptions)/meshes/px100_meshes/gripper_finger.stl"
+            filename="file://$(find interbotix_xsarm_descriptions)/meshes/px100_meshes/gripper_finger.stl"
             scale="0.001 0.001 0.001"
           />
